File: PTP_Project1_Dovsak/PTP_Project1_Dovsak.kicad_pcb (KiCad board)
At the start: 2 copper layers, 45 parts, among them U1 LM2574N-5, U2 4027, U3 4027, U4 74LS47, U5 NE555P, U6 SN74LVC1G11, U7 SA39-12EWA

Commit message: LV8_gotova
LV 8 je gotova
Parts:
- moved R20 86.9 mm to (162.2, 113.2), turned to 90 degrees
- moved R19 86.8 mm to (162.0, 107.0), turned to 90 degrees
- moved C1 72.1 mm to (175.5, 71.0), turned to 90 degrees
- moved U6 62.2 mm to (186.4, 101.0)
- moved C2 61.8 mm to (196.5, 76.5), turned to 90 degrees
- moved SW1 61.4 mm to (202.8, 132.8)
- moved C3 60.2 mm to (195.8, 123.8), turned to 90 degrees
- moved R8 57.6 mm to (235.9, 110.8)
- moved R5 57.5 mm to (235.9, 104.8)
- moved R6 57.5 mm to (235.9, 107.8)
- moved J1 57.4 mm to (167.5, 89.0), turned to 90 degrees
- moved R13 50.1 mm to (198.8, 123.8), turned to 90 degrees
- moved R10 50.0 mm to (207.0, 123.7), turned to 90 degrees
- moved L1 49.9 mm to (197.0, 86.5), turned to 90 degrees
- moved R11 45.3 mm to (209.8, 123.7), turned to 90 degrees
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- renumbered U7 to U5, U5 to U7
Routing:
- net +5V: track 0.00 -> 206.8 mm, vias 0 -> 13
- net Q3: track 0.00 -> 68.7 mm, vias 0 -> 6
- net Q0: track 0.00 -> 64.7 mm, vias 0 -> 4
- net GND: track 0.00 -> 52.8 mm, vias 0 -> 5
- net Q1: track 0.00 -> 48.8 mm, vias 0 -> 2
- net Clock: track 0.00 -> 47.5 mm, vias 0 -> 2
- net Reset: track 0.00 -> 35.3 mm, vias 0 -> 2
- net Q2: track 0.00 -> 33.9 mm, vias 0 -> 4
- net Net-(U7-DIS): track 0.00 -> 33.6 mm
- net Net-(D4-K): track 0.00 -> 30.6 mm
- net Net-(SW2-C): track 0.00 -> 27.6 mm
- net VD: track 0.00 -> 26.9 mm
- net Net-(U4-BI): track 0.00 -> 26.5 mm
- net Net-(U7-THR): track 0.00 -> 24.9 mm, vias 0 -> 2
- net Net-(U2A-J): track 0.00 -> 22.5 mm
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- added copper zone on B.Cu, net GND

Commit message: Gotova LV potpuno
Parts:
- moved R12 0.59 mm to (212.5, 123.7)
Routing:
- net +5V: track 206.8 -> 219.5 mm
- net Net-(SW2-C): track 27.6 -> 30.6 mm
- net Net-(U7-THR): track 24.9 -> 25.5 mm
- net Q1: track 48.8 -> 49.0 mm, vias 2 -> 1
Other:
- board outline added: 100 x 80 mm
- board text added: "Leon Dovšak"
