File: PTP_Project1_Dovsak/PTP_Project1_Dovsak.kicad_sch (KiCad schematic)
At the start: 2 parts

Commit message: LV2 rijesen
Parts:
- removed R1, R3: R_Small, symbol Device:R_Small
- added C3: 22u, symbol Device:C_Polarized
- added C4: 1u, symbol Device:C
- added C6: 220u, symbol Device:C_Polarized
- added C7: 10u, symbol Device:C
- added CB: 100n, symbol Device:C
- added D1: 11DQO6, symbol Device:D_Schottky_Filled
- added D2, D3, D4, D5: (no value), symbol Device:LED
- added J1: ~, symbol Connector:Screw_Terminal_01x02
- added L1: 330u, symbol Device:L
- added R1, R2: 2k, symbol Device:R
- added R3, R4: 47k, symbol Device:R
- added R6, R7, R8, R9: 4k7, symbol Device:R
- added SW1: ~, symbol Switch:SW_Push
- added SW2: ~, symbol Switch:SW_SPDT_312
- added U2: LM2574N-5, Package_DIP:DIP-8_W7.62mm, symbol Regulator_Switching:LM2574N-5
- added U5: NE555P, Package_DIP:DIP-8_W7.62mm, symbol Timer:NE555P
Connections:
- net GND: now also C3.2, C4.1, C6.2, C7.2, CB.2, D1.2 (A), J1.1 (Pin_1), R6.2, R7.2, R8.2, R9.2, SW1.1, U2.2 (SGND), U2.3 (~{ON}/OFF), U2.4 (PGND), U5.1 (GND)
- new net: D3.1 (K), R7.1
- new net: R3.2, R4.1, U5.7 (DIS)
- new net: C7.1, R4.2, U5.2 (TR), U5.6 (THR)
- new net: D4.1 (K), R8.1
- new net: C4.2, R1.2, R2.2, SW2.3 (C)
- new net: R2.1, SW1.2
- new net: D1.1 (K), L1.1, U2.7 (OUT)
- new net: D5.1 (K), R9.1
- new net: D2.1 (K), R6.1
- new net +5V: C6.1, CB.1, L1.2, R1.1, R3.1, U2.1 (FB), U5.4 (R), U5.8 (VCC)
- new net 555: SW2.2 (A), U5.3 (Q)
- new net Clock: SW2.1 (B)
- new net Q0: D2.2 (A)
- new net Q1: D3.2 (A)
- new net Q2: D4.2 (A)
- new net Q3: D5.2 (A)
- new net VD: C3.1, J1.2 (Pin_2), U2.5 (VIN)

Commit message: LV3
Zavrsena VL3
Parts:
- added U6: SN74LVC1G11, SOT-23-6:SOT-23-6, symbol SN74LVC1G11:SN74LVC1G11
- D1: renamed from D2; value (none) -> ~
- D2: renamed from D3; value (none) -> ~
- D3: renamed from D4; value (none) -> ~
- D5: value (none) -> ~
- renumbered C3 to C1, C6 to C2, C4 to C3, CB to C4, C7 to C5, D1 to D4, R6 to R1, R2 to R13, R3 to R19, R7 to R2, R4 to R20, R8 to R3, R9 to R4, R1 to R7
Connections:
- net +5V: now also U6.5 (VCC)
- net Clock: now also R7.2, U6.6 (C)
- net GND: now also U6.2 (GND)
- net Q1: now also U6.1 (A)
- net Q3: now also U6.3 (B)
- net at C3.2, R13.2, SW2.3 (C): no longer R7.2
- new net Reset: U6.4 (Y)
Other:
- moved on the sheet: C1, C2, C3, D1, D2, D3, D4, D5, J1, L1, R1, R2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

Commit message: LV4 rijesen
zavrsena lv4
Parts:
- removed U2: LM2574N-5, Package_DIP:DIP-8_W7.62mm, symbol Regulator_Switching:LM2574N-5
- added H1, H2, H3, H4: MountingHole, symbol Mechanical:MountingHole
- added R10, R11, R12, R9: 10k, symbol Device:R
- added R14, R16, R17, R18, R5, R6, R8: 2k, symbol Device:R_Small
- added R15: R, symbol Device:R
- added U1: LM2574N-5, Package_DIP:DIP-8_W7.62mm_Socket_LongPads, symbol Regulator_Switching:LM2574N-5
- added U2, U3: 4027, Package_DIP:DIP-16_W7.62mm_Socket_LongPads, symbol 4xxx:4027
- added U4: 74LS47, symbol 74xx:74LS47
- added U7: SA39-12EWA, Display_7Segment:Sx39-1xxxxx, symbol Display_Character:SA39-12EWA
Connections:
- net +5V: now also R10.1, R11.1, R12.1, R15.2, R9.1, U1.1 (FB), U2.16 (VDD), U3.16 (VDD), U4.16 (VCC), U7.1 (CA), U7.6 (CA)
- net Clock: now also U2.3 (C)
- net GND: now also U1.2 (SGND), U1.3 (~{ON}/OFF), U1.4 (PGND), U2.7 (R), U2.8 (VSS), U2.9 (R), U3.7 (R), U3.8 (VSS), U3.9 (R), U4.8 (GND)
- net Q0: now also U2.1 (Q), U2.13 (C), U4.7 (A)
- net Q1: now also U2.15 (Q), U3.3 (C), U4.1 (B)
- net Q2: now also U3.1 (Q), U3.13 (C), U4.2 (C)
- net Q3: now also U3.15 (Q), U4.6 (D)
- net Reset: now also U2.12 (S), U2.4 (S), U3.12 (S), U3.4 (S)
- net VD: now also U1.5 (VIN)
- net at D4.1 (K), L1.1: now also U1.7 (OUT)
- new net: R5.1, U4.13 (a)
- new net: R5.2, U7.10 (A)
- new net: R11.2, U3.5 (J), U3.6 (K)
- new net: R17.1, U4.15 (f)
- new net: R17.2, U7.2 (F)
- new net: R9.2, U2.5 (J), U2.6 (K)
- new net: R18.2, U7.3 (G)
- new net: R16.2, U7.4 (E)
- new net: R14.2, U7.5 (D)
- new net: R8.2, U7.8 (C)
- new net: R6.2, U7.9 (B)
- new net: R6.1, U4.12 (b)
- new net: R14.1, U4.10 (d)
- new net: R8.1, U4.11 (c)
- new net: R18.1, U4.14 (g)
- new net: R15.1, U4.3 (LT), U4.4 (BI), U4.5 (RBI)
- new net: R16.1, U4.9 (e)
- new net: R10.2, U2.10 (K), U2.11 (J)
- new net: R12.2, U3.10 (K), U3.11 (J)
- no-connect marks 1 -> 6
Other:
- note added: "555 timer"
- note added: "JK bistabil"
- note added: "LED diode"
- note added: "Montažne rupe"
- note added: "Napajanje"
- note added: "Napajanje bistabila"
- note added: "Reset brojač"
- note added: "Tipka i ulaz radnog takta"
- moved on the sheet: C1, C2, C3, C4, C5, D1, D2, D3, D4, D5, J1, L1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

Commit message: LV 5 rijesen
Parts:
- C1, C2: footprint (none) -> Capacitor_THT:CP_Radial_D5.0mm_P2.00mm
- C3, C4, C5: footprint (none) -> Capacitor_SMD:C_1206_3216Metric_Pad1.33x1.80mm_HandSolder
- D1, D2, D3, D5: footprint (none) -> LED_THT:LED_D5.0mm
- D4: footprint (none) -> Diode_THT:D_DO-41_SOD81_P12.70mm_Horizontal
- H1, H2, H3, H4: footprint (none) -> MountingHole:MountingHole_5.5mm
- J1: footprint (none) -> TerminalBlock_MetzConnect:TerminalBlock_MetzConnect_Type011_RT05502HBLC_1x02_P5.00mm_Horizontal
- L1: footprint (none) -> Inductor_THT:L_Radial_D7.2mm_P3.00mm_Murata_1700
- R1, R2, R3, R4: footprint (none) -> Resistor_THT:R_Axial_DIN0207_L6.3mm_D2.5mm_P10.16mm_Horizontal
- R10, R11, R12, R13, R14, R15, R16, R17, R18, R19, R20, R5, R6, R7, R8, R9: footprint (none) -> Resistor_SMD:R_1206_3216Metric_Pad1.30x1.75mm_HandSolder
- SW1: footprint (none) -> Button_Switch_THT:SW_PUSH_6mm_H4.3mm
- SW2: footprint (none) -> Button_Switch_THT:SW_Slide_SPDT_Straight_CK_OS102011MS2Q
- U4: footprint (none) -> Package_DIP:DIP-16_W7.62mm_Socket_LongPads
- U6: footprint SOT-23-6:SOT-23-6 -> Package_TO_SOT_SMD:SOT-23-6
- U7: footprint Display_7Segment:Sx39-1xxxxx -> Display_7Segment:HDSP-7401
Changed lines of the file:
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@@
 			)
 		)
-		(property "Footprint" ""
+		(property "Footprint" "Resistor_SMD:R_1206_3216Metric_Pad1.30x1.75mm_HandSolder"
 			(at 246.634 87.122 0)
 			(effects
@@
 			)
 		)
-		(property "Footprint" ""
+		(property "Footprint" "MountingHole:MountingHole_5.5mm"
 			(at 238.76 145.288 0)
 			(effects
@@
 			)
 		)
-		(property "Footprint" ""
+		(property "Footprint" "Resistor_SMD:R_1206_3216Metric_Pad1.30x1.75mm_HandSolder"
 			(at 246.634 112.522 0)
 			(effects
@@
 			)
 		)
-		(property "Footprint" ""
+		(property "Footprint" "Resistor_THT:R_Axial_DIN0207_L6.3mm_D2.5mm_P10.16mm_Horizontal"
 			(at 262.89 38.608 90)
 			(effects
@@
 			)
 		)
-		(property "Footprint" ""
+		(property "Footprint" "Resistor_SMD:R_1206_3216Metric_Pad1.30x1.75mm_HandSolder"
 			(at 101.092 105.918 90)
 			(effects
@@
 			)
 		)
-		(property "Footprint" ""
+		(property "Footprint" "LED_THT:LED_D5.0mm"
 			(at 246.38 43.18 0)
 			(effects
@@
 			)
 		)
-		(property "Footprint" "Display_7Segment:Sx39-1xxxxx"
+		(property "Footprint" "Display_7Segment:HDSP-7401"
 			(at 272.034 118.872 0)
 			(effects
@@
 			)
 		)
-		(property "Footprint" ""
+		(property "Footprint" "Resistor_THT:R_Axial_DIN0207_L6.3mm_D2.5mm_P10.16mm_Horizontal"
 			(at 262.89 44.958 90)
 			(effects
@@
 			)
 		)
-		(property "Footprint" ""
+		(property "Footprint" "Capacitor_SMD:C_1206_3216Metric_Pad1.33x1.80mm_HandSolder"
 			(at 103.8352 123.698 0)
 			(effects
@@
 			)
 		)
-		(property "Footprint" ""
+		(property "Footprint" "Resistor_SMD:R_1206_3216Metric_Pad1.30x1.75mm_HandSolder"
 			(at 21.082 161.29 90)
 			(effects
@@
 			)
 		)
-		(property "Footprint" ""
+		(property "Footprint" "Resistor_SMD:R_1206_3216Metric_Pad1.30x1.75mm_HandSolder"
 			(at 246.634 92.202 0)
 			(effects
@@
 			)
 		)
-		(property "Footprint" ""
+		(property "Footprint" "Capacitor_SMD:C_1206_3216Metric_Pad1.33x1.80mm_HandSolder"
 			(at 40.894 90.4748 0)
 			(effects
@@
 			)
 		)
-		(property "Footprint" ""
+		(property "Footprint" "Resistor_SMD:R_1206_3216Metric_Pad1.30x1.75mm_HandSolder"
 			(at 45.974 107.188 90)
 			(effects
@@
 			)
 		)
-		(property "Footprint" ""
+		(property "Footprint" "Capacitor_THT:CP_Radial_D5.0mm_P2.00mm"
 			(at 47.1932 50.292 0)
 			(effects
@@
 			)
 		)
-		(property "Footprint" ""
+		(property "Footprint" "Resistor_THT:R_Axial_DIN0207_L6.3mm_D2.5mm_P10.16mm_Horizontal"
 			(at 262.89 51.308 90)
 			(effects
@@
 			)
 		)
-		(property "Footprint" ""
+		(property "Footprint" "LED_THT:LED_D5.0mm"
 			(at 246.38 30.48 0)
 			(effects
@@
 			)
 		)
-		(property "Footprint" ""
+		(property "Footprint" "Diode_THT:D_DO-41_SOD81_P12.70mm_Horizontal"
 			(at 89.408 47.752 0)
 			(effects
@@
 			)
 		)
-		(property "Footprint" ""
+		(property "Footprint" "Package_DIP:DIP-16_W7.62mm_Socket_LongPads"
 			(at 218.694 104.902 0)
 			(effects
@@
 			)
 		)
-		(property "Footprint" ""
+		(property "Footprint" "MountingHole:MountingHole_5.5mm"
 			(at 238.76 160.528 0)
 			(effects
@@
 			)
 		)
-		(property "Footprint" ""
+		(property "Footprint" "Resistor_SMD:R_1206_3216Metric_Pad1.30x1.75mm_HandSolder"
 			(at 246.634 97.282 0)
 			(effects
@@
 			)
 		)
-		(property "Footprint" ""
+		(property "Footprint" "Resistor_SMD:R_1206_3216Metric_Pad1.30x1.75mm_HandSolder"
 			(at 246.634 107.442 0)
 			(effects
@@
 			)
 		)
-		(property "Footprint" ""
+		(property "Footprint" "Inductor_THT:L_Radial_D7.2mm_P3.00mm_Murata_1700"
 			(at 97.028 37.592 0)
 			(effects
@@
 			)
 		)
-		(property "Footprint" ""
+		(property "Footprint" "Resistor_SMD:R_1206_3216Metric_Pad1.30x1.75mm_HandSolder"
 			(at 101.092 84.328 90)
 			(effects
@@
 			)
 		)
-		(property "Footprint" ""
+		(property "Footprint" "Resistor_SMD:R_1206_3216Metric_Pad1.30x1.75mm_HandSolder"
 			(at 49.022 160.02 90)
 			(effects
@@
 			)
 		)
-		(property "Footprint" ""
+		(property "Footprint" "Resistor_THT:R_Axial_DIN0207_L6.3mm_D2.5mm_P10.16mm_Horizontal"
 			(at 262.89 32.258 90)
 			(effects
@@
 			)
 		)
-		(property "Footprint" ""
+		(property "Footprint" "Resistor_SMD:R_1206_3216Metric_Pad1.30x1.75mm_HandSolder"
 			(at 246.634 102.362 0)
 			(effects
@@
 			)
 		)
-		(property "Footprint" ""
+		(property "Footprint" "LED_THT:LED_D5.0mm"
 			(at 246.38 36.83 0)
 			(effects
@@
 			)
 		)
-		(property "Footprint" ""
+		(property "Footprint" "Resistor_SMD:R_1206_3216Metric_Pad1.30x1.75mm_HandSolder"
 			(at 188.976 109.982 90)
 			(effects
@@
 			)
 		)
-		(property "Footprint" ""
+		(property "Footprint" "Resistor_SMD:R_1206_3216Metric_Pad1.30x1.75mm_HandSolder"
 			(at 78.486 97.79 90)
 			(effects
@@
 			)
 		)
-		(property "Footprint" ""
+		(property "Footprint" "Resistor_SMD:R_1206_3216Metric_Pad1.30x1.75mm_HandSolder"
 			(at 74.422 160.02 90)
 			(effects
@@
 			)
 		)
-		(property "Footprint" ""
+		(property "Footprint" "Button_Switch_THT:SW_PUSH_6mm_H4.3mm"
 			(at 33.274 100.33 0)
 			(effects
@@
 			)
 		)
-		(property "Footprint" ""
+		(property "Footprint" "MountingHole:MountingHole_5.5mm"
 			(at 238.76 152.908 0)
 			(effects
@@
 			)
 		)
-		(property "Footprint" ""
+		(property "Footprint" "Resistor_SMD:R_1206_3216Metric_Pad1.30x1.75mm_HandSolder"
 			(at 98.552 160.02 90)
 			(effects
@@
 			)
 		)
-		(property "Footprint" ""
+		(property "Footprint" "Resistor_SMD:R_1206_3216Metric_Pad1.30x1.75mm_HandSolder"
 			(at 246.634 117.602 0)
 			(effects
@@
 			)
 		)
-		(property "Footprint" ""
+		(property "Footprint" "MountingHole:MountingHole_5.5mm"
 			(at 238.76 137.668 0)
 			(effects
@@
 			)
 		)
-		(property "Footprint" ""
+		(property "Footprint" "TerminalBlock_MetzConnect:TerminalBlock_MetzConnect_Type011_RT05502HBLC_1x02_P5.00mm_Horizontal"
 			(at 20.828 41.402 0)
 			(effects
@@
 			)
 		)
-		(property "Footprint" ""
+		(property "Footprint" "LED_THT:LED_D5.0mm"
 			(at 246.38 49.53 0)
 			(effects
@@
 			)
 		)
-		(property "Footprint" ""
+		(property "Footprint" "Capacitor_THT:CP_Radial_D5.0mm_P2.00mm"
 			(at 113.2332 51.562 0)
 			(effects
@@
 			)
 		)
-		(property "Footprint" "SOT-23-6:SOT-23-6"
+		(property "Footprint" "Package_TO_SOT_SMD:SOT-23-6"
 			(at 183.896 139.446 0)
 			(effects
@@
 			)
 		)
-		(property "Footprint" ""
+		(property "Footprint" "Button_Switch_THT:SW_Slide_SPDT_Straight_CK_OS102011MS2Q"
 			(at 70.104 97.79 0)
 			(effects
@@
 			)
 		)
-		(property "Footprint" ""
+		(property "Footprint" "Capacitor_SMD:C_1206_3216Metric_Pad1.33x1.80mm_HandSolder"
 			(at 119.3292 87.63 0)
 			(effects

Commit message: Gotova LV potpuno
Parts:
- renumbered U7 to U5, U5 to U7
Changed lines of the file:
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@@
 		(dnp no)
 		(fields_autoplaced yes)
-		(property "Reference" "U7"
-			(at 272.034 87.122 0)
+		(property "Reference" "U5"
+			(at 272.034 87.63 0)
 			(effects
 				(font
@@
 		)
 		(property "Value" "SA39-12EWA"
-			(at 272.034 89.662 0)
+			(at 272.034 90.17 0)
 			(effects
 				(font
@@
 			(project ""
 				(path "/b0353478-dd11-49a7-a92d-64a8149990f5"
-					(reference "U7")
+					(reference "U5")
 					(unit 1)
 				)
@@
 		(on_board yes)
 		(dnp no)
-		(property "Reference" "U5"
+		(property "Reference" "U7"
 			(at 145.288 84.074 0)
 			(effects
@@
 			(project ""
 				(path "/b0353478-dd11-49a7-a92d-64a8149990f5"
-					(reference "U5")
-					(unit 1)
-				)
+					(reference "U7")
+					(unit 1)
+				)
